File: rev01/usbhub_c4.kicad_pcb (KiCad board)
At the start: 4 copper layers, 45.8 x 45.8 mm, 118 parts, among them J1 5077CR-16SMC2, J2 Conn_01x01, J3 5077CR-16SMC2, J4 5077CR-16SMC2, J5 5077CR-16SMC2, J6 5077CR-16SMC2, J7 Conn_01x01, J8 Conn_01x01, Q1 BSS138, Q2 BSS138, Q3 BSS138, Q4 BSS138, U1 TPS25821, U2 LM3670MF-3.3, U3 TPS25821, U4 μPD720115, U5 TPS25821, U6 TPS25821, Y1 24MHz

Commit message: シンプル版追加
Parts:
- added SW1: SKRPACE010, _platinumegg:SW_Push_1P1T_alps_SKRP, F.Cu at (111.9, 82.1)
- renumbered C30 to C1, C5 to C10, C26 to C11, C27 to C12, C28 to C13, C18 to C14, C19 to C15, C20 to C16, C7 to C17, C8 to C18, C9 to C19, C29 to C2, C10 to C20, C6 to C21, C12 to C22, C13 to C23, C14 to C24, C15 to C25, C11 to C26, C31 to C27, C32 to C28, C33 to C29, C38 to C3, C34 to C30, C23 to C31, C2 to C32, C3 to C33, C35 to C34, C36 to C35, C1 to C36, C37 to C4, C16 to C5, C17 to C6, C22 to C7, C21 to C8, C25 to C9, D7 to D10, D12 to D11, D13 to D12, D15 to D13, D16 to D14, D17 to D15, D18 to D16, D3 to D2, D2 to D3, D14 to D4, D8 to D5, D9 to D6, D10 to D7, D11 to D8, D6 to D9, FB2 to FB1, J7 to J3, J8 to J4, J3 to J5, J4 to J6, J5 to J7, J6 to J8, R7 to R1, R13 to R10, R20 to R11, R21 to R12, R22 to R13, R24 to R14, R11 to R15, R1 to R16, R4 to R17, R5 to R18, R14 to R19, R8 to R2, R34 to R20, R10 to R21, R15 to R22, R18 to R23, R16 to R24, R17 to R25, R23 to R26, R30 to R27, R33 to R28, R31 to R29, R2 to R3, R32 to R30, R37 to R31, R38 to R32, R41 to R33, R39 to R34, R40 to R35, R3 to R36, R42 to R37, R45 to R38, R43 to R39, R19 to R4, R44 to R40, R36 to R5, R35 to R6, R6 to R7, R9 to R8, R12 to R9, U2 to U1, U4 to U2, U5 to U4, U6 to U5, U1 to U6
Routing:
- net /~{RESET}: track 9.58 -> 49.6 mm, vias 0 -> 2
- net GND: track 93.9 -> 98.1 mm
Other:
- board text added: "Kmnabrm USBHUB"
- board text added: "Reset SW"
- board text added: "rev 0.1.1@2025-05-11"
- board text removed: "April 28, 2025 rev 0.1.0"
- board text removed: "Kmnabrm makes all the difference."
